File: hardware/KiCad/THT/original/quasimodo_tht_orig.kicad_pcb (KiCad board)
At the start: 2 copper layers, 97 x 46 mm, 41 parts, among them J1 +Vin, J2 +Vin, J3 GND, J4 GND, J5 scope, J6 scope GND, J7 Screw_Terminal_01x02, Q1 NTD4906, SW1 SW_DIP_x04, U1 LMC555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

Commit message: Add files via upload
Parts:
- Cs_1, Cx_1: value PinSocket_2x03_P2.54mm_Vertical_no_silk -> Preci-Dip_2x03_P2.54mm_Vertical_no_silk; footprint analoghifi:PinSocket_2x03_P2.54mm_Vertical_no_silk -> analoghifi:Preci-Dip_2x03_P2.54mm_Vertical_no_silk
- Cs_2, Cx_2: value PinSocket_2x04_P2.54mm_Vertical_no_silk -> Preci-Dip_2x04_P2.54mm_Vertical_no_silk; footprint analoghifi:PinSocket_2x04_P2.54mm_Vertical_no_silk -> analoghifi:Preci-Dip_2x04_P2.54mm_Vertical_no_silk
- Rs: value PinSocket_1x03_P2.54mm_Vertical_no_silk -> Preci-Dip_1x03_P2.54mm_Vertical_no_silk; footprint analoghifi:PinSocket_1x03_P2.54mm_Vertical_no_silk -> analoghifi:Preci-Dip_1x03_P2.54mm_Vertical_no_silk
