File: hardware/KiCad/THT/original/quasimodo_tht_orig.kicad_sch (KiCad schematic)
At the start: 35 parts, among them J1 +Vin, J2 +Vin, J3 GND, J4 GND, J5 scope, J6 scope GND, J7 Screw_Terminal_01x02, Q1 NTD4906, SW1 SW_DIP_x04, U1 LMC555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

Commit message: Add files via upload
Parts:
- RV1: value (none) -> 1kΩ
Other:
- note added: "(DIP-Sw. 2 and 3 always open / not needed)"
- note added: "1"
- note added: "2"
- note added: "3"
- note added: "4"
- note added: "DIP-Sw. 1 4 R fosc 0 0 39k ~120Hz 1 0 7.96k ~600Hz 0 1 1.9k ~2500Hz 1 1 1.6k ~2980Hz"
- note added: "U1 can be LMC555 or TLC555 or ICM7555(IPAZ) or even a different type important: it has to be a 555 timer in CMOS technology (with rail-to-rail output swing)"
- note added: "stimulus frequency fosc = 1/(1.4*R*C4)"
Changed lines of the file:
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@@
+    (stroke (width 0) (type default) (color 0 0 0 0))
+  )
+  (polyline (pts (xy 71.7821 155.5986) (xy 71.7821 170.6908))
     (stroke (width 0) (type default) (color 0 0 0 0))
   )
@@
     (stroke (width 0) (type default) (color 0 0 0 0))
   )
-  (wire (pts (xy 168.91 101.6) (xy 168.91 105.41))
+  (wire (pts (xy 168.91 91.44) (xy 168.91 105.41))
     (stroke (width 0) (type default) (color 0 0 0 0))
   )
@@
     (stroke (width 0) (type default) (color 0 0 0 0))
   )
+  (polyline (pts (xy 63.0919 155.652) (xy 63.0927 170.6908))
+    (stroke (width 0) (type solid) (color 0 0 0 0))
+  )
   (wire (pts (xy 95.25 127) (xy 114.3 127))
     (stroke (width 0) (type default) (color 0 0 0 0))
@@
     (stroke (width 0) (type default) (color 0 0 0 0))
   )
+  (polyline (pts (xy 88.9 170.6882) (xy 88.8992 155.6494))
+    (stroke (width 0) (type solid) (color 0 0 0 0))
+  )
   (wire (pts (xy 214.63 43.18) (xy 214.63 48.26))
     (stroke (width 0) (type default) (color 0 0 0 0))
@@
     (stroke (width 0) (type default) (color 0 0 0 0))
   )
+  (polyline (pts (xy 63.5 161.29) (xy 88.9 161.29))
+    (stroke (width 0) (type default) (color 0 0 0 0))
+  )
   (wire (pts (xy 81.28 30.48) (xy 81.28 34.29))
     (stroke (width 0) (type default) (color 0 0 0 0))
@@
     (stroke (width 0) (type default) (color 0 0 0 0))
   )
+  (polyline (pts (xy 71.7821 170.6908) (xy 71.9853 170.6908))
+    (stroke (width 0) (type default) (color 0 0 0 0))
+  )
   (wire (pts (xy 53.34 54.61) (xy 53.34 46.99))
     (stroke (width 0) (type default) (color 0 0 0 0))
@@
     (stroke (width 0) (type default) (color 0 0 0 0))
   )
-  (wire (pts (xy 130.81 109.22) (xy 130.81 101.6))
+  (wire (pts (xy 130.81 109.22) (xy 130.81 91.44))
     (stroke (width 0) (type default) (color 0 0 0 0))
   )
@@
     (stroke (width 0) (type default) (color 0 0 0 0))
   )
+  (polyline (pts (xy 63.0927 170.6908) (xy 88.9 170.6882))
+    (stroke (width 0) (type solid) (color 0 0 0 0))
+  )
   (wire (pts (xy 214.63 30.48) (xy 214.63 35.56))
     (stroke (width 0) (type default) (color 0 0 0 0))
@@
     (stroke (width 0) (type default) (color 0 0 0 0))
   )
+  (polyline (pts (xy 63.0919 155.652) (xy 88.8992 155.6494))
+    (stroke (width 0) (type solid) (color 0 0 0 0))
+  )
   (wire (pts (xy 93.98 127) (xy 95.25 127))
     (stroke (width 0) (type default) (color 0 0 0 0))
@@
   (wire (pts (xy 204.47 43.18) (xy 204.47 48.26))
     (stroke (width 0) (type default) (color 0 0 0 0))
+  )
+  (text "stimulus frequency \nfosc = 1/(1.4*R*C4)" (at 63.5 153.67 0)
+    (effects (font (size 1.27 1.27)) (justify left bottom))
   )
   (text "Cs" (at 203.2 133.35 180)
     (effects (font (size 2.54 2.54)) (justify right bottom))
   )
+  (text "U1 can be LMC555 or TLC555 or ICM7555(IPAZ) or even a different type\nimportant: it has to be a 555 timer in CMOS technology\n(with rail-to-rail output swing)"
+    (at 57.15 80.01 0)
+    (effects (font (size 1.27 1.27)) (justify left bottom))
+  )
+  (text "2" (at 71.8329 138.972 0)
+    (effects (font (size 0.75 0.75)) (justify left bottom))
+  )
+  (text "DIP-Sw.\n 1   4    R      fosc\n\n 0   0   39k     ~120Hz\n 1   0   7.96k   ~600Hz\n 0   1   1.9k   ~2500Hz\n 1   1   1.6k   ~2980Hz"
+    (at 63.5 170.18 0)
+    (effects (font (size 1.27 1.27)) (justify left bottom))
+  )
+  (text "3" (at 71.9068 141.3488 0)
+    (effects (font (size 0.75 0.75)) (justify left bottom))
+  )
   (text "Rs" (at 203.2 143.51 180)
     (effects (font (size 2.54 2.54)) (justify right bottom))
@@
     (effects (font (size 2.54 2.54)) (justify right bottom))
   )
+  (text "(DIP-Sw. 2 and 3 always open / not needed)" (at 62.23 173.99 0)
+    (effects (font (size 1 1)) (justify left bottom))
+  )
+  (text "4" (at 71.983 144.0166 0)
+    (effects (font (size 0.75 0.75)) (justify left bottom))
+  )
+  (text "1" (at 71.8306 136.318 0)
+    (effects (font (size 0.75 0.75)) (justify left bottom))
+  )
   (label "+Vin" (at 55.88 30.48 0)
     (effects (font (size 1.27 1.27)) (justify left bottom))
   )
   (label "DRAIN" (at 184.15 119.38 180)
-    (effects (font (size 1.27 1.27)) (justify right bottom))
+    (effects (font (size 1 1)) (justify right bottom))
   )
   (label "TRAFO" (at 214.63 119.38 180)
-    (effects (font (size 1.27 1.27)) (justify right bottom))
+    (effects (font (size 1 1)) (justify right bottom))
   )
   (label "FETGATE" (at 160.02 127 180)
-    (effects (font (size 1.27 1.27)) (justify right bottom))
+    (effects (font (size 1 1)) (justify right bottom))
   )
   (label "RC_NODE" (at 73.66 127 180)
-    (effects (font (size 1.27 1.27)) (justify right bottom))
+    (effects (font (size 1 1)) (justify right bottom))
   )
   (label "OSC" (at 95.25 97.79 180)
-    (effects (font (size 1.27 1.27)) (justify right bottom))
+    (effects (font (size 1 1)) (justify right bottom))
   )
   (label "Rs_Cs" (at 205.74 135.89 0)
@@
     )
   )
-  (global_label "VCC" (shape input) (at 130.81 101.6 90) (fields_autoplaced)
+  (global_label "VCC" (shape input) (at 130.81 91.44 90) (fields_autoplaced)
     (effects (font (size 1.27 1.27)) (justify left))
-    (property "Intersheet References" "${INTERSHEET_REFS}" (id 0) (at 130.7306 95.5583 90)
+    (property "Intersheet References" "${INTERSHEET_REFS}" (id 0) (at 130.7306 85.3983 90)
       (effects (font (size 1.27 1.27)) (justify left) hide)
     )
@@
     )
   )
-  (global_label "VCC" (shape input) (at 168.91 101.6 90) (fields_autoplaced)
+  (global_label "VCC" (shape input) (at 168.91 91.44 90) (fields_autoplaced)
     (effects (font (size 1.27 1.27)) (justify left))
-    (property "Intersheet References" "${INTERSHEET_REFS}" (id 0) (at 168.8306 95.5583 90)
+    (property "Intersheet References" "${INTERSHEET_REFS}" (id 0) (at 168.8306 85.3983 90)
       (effects (font (size 1.27 1.27)) (justify left) hide)
     )
@@
       (effects (font (size 1.27 1.27)) (justify right))
     )
-    (property "Value" "" (id 1) (at 213.36 142.24 0)
+    (property "Value" "1kΩ" (id 1) (at 213.36 142.24 0)
       (effects (font (size 1.27 1.27)) (justify right))
     )

Commit message: Add files via upload
Other:
- note added: "*"
- note added: "Vcc Power supply +5V to +15V"
- note added: "the LMC555 (from TI) has an "absolute max. VCC" of 15V and the MCP1406/07 (from TI) (or its replacemant type TC4420/TC4429) have a "recommended min. Operating Voltage" of 4.5V"
Changed lines of the file:
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@@
     (effects (font (size 1.27 1.27)) (justify left bottom))
+  )
+  (text "Vcc Power supply +5V to +15V" (at 12.7 34.29 0)
+    (effects (font (size 1.27 1.27)) (justify left bottom))
+  )
+  (text "*" (at 43.5119 34.5941 0)
+    (effects (font (size 2 2)) (justify left bottom))
   )
   (text "Cs" (at 203.2 133.35 180)
@@
     (effects (font (size 0.75 0.75)) (justify left bottom))
   )
+  (text "the LMC555 (from TI) has an \"absolute max. VCC\" of 15V\nand the MCP1406/07 (from TI) (or its replacemant type TC4420/TC4429) \nhave a \"recommended min. Operating Voltage\" of 4.5V"
+    (at 13.97 196.85 0)
+    (effects (font (size 1.27 1.27)) (justify left bottom))
+  )
+  (text "*" (at 12.3717 193.0573 0)
+    (effects (font (size 2 2)) (justify left bottom))
+  )
   (label "+Vin" (at 55.88 30.48 0)
